File: Zx50_Cpu/Zx50_Cpu.kicad_sch (KiCad schematic)
At the start: 24 parts, among them J1 Zx50_EdgeConnector, J2 FrontPanelConnect, J3 Clock Mezzanine, J4 Front Panel, SW1 RESET, U1 74AHC1G14, U2 SN74AHCT245N, U3 SN74AHCT245N, U4 Z84C00xxP, U5 SN74AHCT245N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

Commit message: 4 layer done
Parts:
- J1: footprint Connector_PinSocket_2.54mm:PinSocket_2x40_P2.54mm_Vertical_Oval -> zx50_footprints:PinHeader_2x40_P2.54mm_Horizontal_Edge
- R2: footprint Resistor_THT:R_Axial_DIN0207_L6.3mm_D2.5mm_P10.16mm_Horizontal -> Resistor_THT:R_Axial_DIN0207_L6.3mm_D2.5mm_P5.08mm_Vertical
Changed lines of the file:
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@@
 			)
 		)
-		(property "Footprint" "Resistor_THT:R_Axial_DIN0207_L6.3mm_D2.5mm_P10.16mm_Horizontal"
+		(property "Footprint" "Resistor_THT:R_Axial_DIN0207_L6.3mm_D2.5mm_P5.08mm_Vertical"
 			(at 222.25 96.52 0)
 			(effects
@@
 			)
 		)
-		(property "Datasheet" "~"
+		(property "Datasheet" ""
 			(at 222.25 96.52 0)
 			(effects
@@
 			)
 		)
-		(property "Description" "Resistor, small symbol"
+		(property "Description" ""
 			(at 222.25 96.52 0)
 			(effects
@@
 			)
 		)
-		(property "Footprint" "Connector_PinSocket_2.54mm:PinSocket_2x40_P2.54mm_Vertical_Oval"
+		(property "Footprint" "zx50_footprints:PinHeader_2x40_P2.54mm_Horizontal_Edge"
 			(at 128.524 170.18 0)
 			(effects
@@
 			)
 		)
-		(property "Datasheet" "~"
+		(property "Datasheet" ""
 			(at 73.66 180.34 0)
 			(effects
@@
 			)
 		)
-		(property "Description" "Generic connector, double row, 02x40, odd/even pin numbering scheme (row 1 odd numbers, row 2 even numbers), script generated (kicad-library-utils/schlib/autogen/connector/)"
+		(property "Description" ""
 			(at 131.572 173.736 0)
 			(effects
