File: boards/Zx50_FrontPanelDisplay/Zx50_FrontPanelDisplay.kicad_pcb (KiCad board)
At the start: 2 copper layers, 152.4 x 114.3 mm, 41 parts, among them J1 Front Panel 2, J2 Front Panel, J3 Remote Off, SW1 DISP_EN, SW2 RUN, SW3 STEP, SW4 RESET, SW5 POWER, U1 HCMS-3973, U2 SN74HC595N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

Commit message: reorg documentation.
Parts:
- removed H3, H4: MountingHole, MountingHole:MountingHole_3.2mm_M3
Routing:
- net Net-(J2-Pin_7): track 165.5 -> 160.6 mm
- net +3.3V: track 498.2 -> 497.6 mm
Other:
- board text added: "ADDRESS"
- board text added: "DATA"
- board text added: "Display Conn"
- board text added: "Remote Power"
- board text added: "STATUS"
- board text added: "Switch Conn"
- board text added: "Zx50 Front Panel Display Marc Mosko, 2026 Zx50_FrontPanelDisplay"
