File: boards/Zx50_Bus_Probe_RevA/Zx50 Bus Probe_RevA.kicad_sch (KiCad schematic)
At the start: 81 parts, among them J1 Zx50_EdgeConnector, J10 CH1, J11 CH2, J12 CH3, J13 DISPL SOCKET, J14 DISPL SOCKET, J15 Z80_Addr, J16 Z80_Data, J17 Z80_Ctrl, J18 Clock, J19 SH_Data, J2 OUT, J20 SH_Ctrl, J3 IN, J4 PIC PGM, J5 P0, J6 P1, J7 P2, J8 Send/Recv Card, J9 CH0, U1 MCP23S17_SP, U10 CD74HC4051E, U11 CD74HC4051E, U12 CD74HC4051E, U13 MCP23S17_SP, U14 CD74HC154M96, U15 OPA356xxD, U16 OPA356xxD, U17 PIC18F4620-I_P, U18 74AHCT541, U19 Jumper, U2 CD74HC4051E, U20 Jumper, U21 Jumper, U22 Jumper, U23 Jumper, U24 Jumper, U25 Jumper, U3 CD74HC4051E, U4 CD74HC4051E, U5 CD74HC4051E, U6 SN74ABT245BN, U7 SN74ABT245BN, U8 CD74HC4051E, U9 CD74HC4051E

Commit message: Many updates and board revisions.
- Backplane Rev D for better AC termination.
- BusProbe revision, much smaller card, use surface mount, faster multiplexers.
- Revised clock mezzanine to reduce ringing.
Parts:
- U10, U11, U12, U2, U3, U4, U5, U8, U9: now fitted
Changed lines of the file:
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@@
 		(in_bom yes)
 		(on_board yes)
-		(dnp yes)
+		(dnp no)
 		(property "Reference" "U4"
 			(at 214.376 324.104 0)
@@
 		(in_bom yes)
 		(on_board yes)
-		(dnp yes)
+		(dnp no)
 		(property "Reference" "U3"
 			(at 213.868 270.51 0)
@@
 		(in_bom yes)
 		(on_board yes)
-		(dnp yes)
+		(dnp no)
 		(property "Reference" "U11"
 			(at 410.7881 300.99 0)
@@
 		(in_bom yes)
 		(on_board yes)
-		(dnp yes)
+		(dnp no)
 		(fields_autoplaced yes)
 		(property "Reference" "U5"
@@
 		(in_bom yes)
 		(on_board yes)
-		(dnp yes)
+		(dnp no)
 		(property "Reference" "U12"
 			(at 408.94 335.28 0)
@@
 		(in_bom yes)
 		(on_board yes)
-		(dnp yes)
+		(dnp no)
 		(property "Reference" "U8"
 			(at 354.33 236.22 0)
@@
 		(in_bom yes)
 		(on_board yes)
-		(dnp yes)
+		(dnp no)
 		(property "Reference" "U10"
 			(at 354.076 325.12 0)
@@
 		(in_bom yes)
 		(on_board yes)
-		(dnp yes)
+		(dnp no)
 		(property "Reference" "U2"
 			(at 212.852 237.744 0)
@@
 		(in_bom yes)
 		(on_board yes)
-		(dnp yes)
+		(dnp no)
 		(property "Reference" "U9"
 			(at 354.33 269.24 0)
