File: boards/Zx50_MemoryCard_RevA1/Zx50_MemoryCard_RevA1.kicad_pcb (KiCad board)
At the start: 4 copper layers, 123.4 x 129.8 mm, 53 parts, among them J1 Zx50_EdgeConnector, J2 JTAG, SW1 SW_DIP_x05, U1 SN74ABT541BN, U10 CY7C1049GN, U11 CY7C1049GN, U12 SST39SF040, U2 74AHCT1G04, U3 SN74ABT16244ADL, U4 74ABT245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

Commit message: fixup pic z80 timing.  add memory test script to pico
Connections:
- J1 pad 42: unconnected-(J1-CLK-Pad42) -> /CLK
- R2 pad 2: Net-(D2-A) -> unconnected-(R2-Pad2)
- U8 pad 90: /CPLD And Memory/~CE0~ -> /CLK
- U8 pad 99: Net-(D2-K) -> /CPLD And Memory/~CE0~
