File: boards/Zx50_Clock_Mezzanine_RevB/Zx50_Clock_Mezzanine_RevB.kicad_sch (KiCad schematic)
At the start: 38 parts, among them J2 Conn_02x05_Odd_Even, J3 Conn_Coaxial, U1 74VHC1G14, U10 74VHC1G14, U2 74AHC74, U3 74AHC1G08, U4 74AHC1G79, U5 74AHC1G32, U6 CD74AC161M96, U7 74VHC125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

Commit message: Lots of updates: Work on memory card Rev C with Lattice XO3LF, finish up the front panel card firmware for the pico., add some results for the clock mezzanine Rev B.
Parts:
- C1, C10, C11, C12, C13, C2, C3, C4, C5, C6, C7, C8: Mouser_PN (none) -> 603-CC805KRX7R9BB104; SKU (none) -> CC0805KRX7R9BB104
- R1, R2: Mouser_PN (none) -> 603-RC0805FR-0710KL; SKU (none) -> RC0805FR-0710KL
- R10, R11, R4, R5, R6, R7, R8, R9: Mouser_PN (none) -> 603-RC0805FR-0733RL; SKU (none) -> RC0805FR-0733RL
- R3: Mouser_PN (none) -> 603-RC0805FR-0749K9L; SKU (none) -> RC0805FR-0749K9L
- U1, U10, U8, U9: Mouser_PN (none) -> 863-MC74VHC1G14DBVTG
- U2: Mouser_PN (none) -> 595-SN74AHC74DR
- U3: Mouser_PN (none) -> 595-SN74AHC1G08DBVR
- U4: Mouser_PN (none) -> 771-AHC1G79GV125
- U5: Mouser_PN (none) -> 595-SN74AHC1G32DBVR
- U6: Mouser_PN (none) -> 595-CD74AC161M96
- U7: Mouser_PN (none) -> 863-MC74VHC125DR2G
