File: boards/Zx50_Backplane_RevD/Zx50_Backplane_RevD.kicad_sch (KiCad schematic)
At the start: 75 parts, among them CN1 100pF, CN10 100pF, CN11 100pF, CN12 100pF, CN13 100pF, CN14 100pF, CN15 100pF, CN16 100pF, CN2 100pF, CN3 100pF, CN4 100pF, CN5 100pF, CN6 100pF, CN7 100pF, CN8 100pF, CN9 100pF, J1 Conn_02x40_Odd_Even, J10 GPIO SEL, J11 POWER, J2 Conn_02x40_Odd_Even, J3 Conn_02x40_Odd_Even, J4 Conn_02x40_Odd_Even, J5 Conn_02x40_Odd_Even, J6 Conn_02x40_Odd_Even, J7 Conn_02x40_Odd_Even, J8 Conn_02x40_Odd_Even

Commit message: pico async is ok, merge to master.  Also add recent work on hw boards
Parts:
- removed CN10, CN11, CN12, CN13, CN14, CN15, CN16, CN2, CN3, CN4, CN5, CN6, CN7, CN8, CN9: 100pF, zx50_footprints:CAP_CA0612_3P2X1P6_YAG, symbol Device:C_Network04
- added CN10, CN11, CN12, CN13, CN14, CN15, CN16, CN2, CN3, CN4, CN5, CN6, CN7, CN8, CN9: 47pF, zx50_footprints:CAP_CA0612_3P2X1P6_YAG, symbol zx50_symbols:CN_47pf_1206x4
- C1, D1, H1, H2, H3, H4, H5, H6, J10, J11: now not fitted
- C10, C12, C13, C14: value 100pF -> 47pF; footprint Capacitor_SMD:C_0805_2012Metric_Pad1.18x1.45mm_HandSolder -> Capacitor_SMD:C_0805_2012Metric; symbol Device:C -> zx50_symbols:C_47pF_0805; LCSC C2167185 -> C14857; SKU C0805C101J5GACTU -> CL21C470JBANNNC
- C2, C3, C4, C5, C6, C7, C8, C9: footprint Capacitor_SMD:C_0805_2012Metric_Pad1.18x1.45mm_HandSolder -> Capacitor_SMD:C_0805_2012Metric; symbol Device:C -> zx50_symbols:C_100nF_0805; LCSC C3018562 -> C28233; SKU C0805C104K5RACTU -> CL21B104KCFNNNE
- CN1: value 100pF -> 47pF; symbol Device:C_Network04 -> zx50_symbols:CN_47pf_1206x4; DigiKey_PN 13-CA0612JRNPO9BN101CT-ND -> 13-CA0612JRNPO9BN470CT-ND; LCSC C1322399 -> C22446551; SKU CA0612JRNPO9BN101 -> CA0612JRNPO9BN470
- J1, J2, J3, J4, J5, J6, J7, J8: now not fitted; now left out of the parts list
- R10, R2, R3, R8, R9: value 100 -> 100R; footprint Resistor_SMD:R_0805_2012Metric_Pad1.20x1.40mm_HandSolder -> Resistor_SMD:R_0805_2012Metric; symbol Device:R -> zx50_symbols:R_100R_100mW_0805; LCSC C105577 -> C17408; SKU RC0805FR-07100RL -> 0805W8F1000T5E
- RN1, RN11, RN13, RN15, RN3, RN4, RN8, RN9: symbol Device:R_Pack08 -> zx50_symbols:RN_100R_SOIC16; LCSC C1357946 -> C1358123; SKU 4816P-1-101LF -> 4816P-T01-101LF
Connections:
- net GND: now also CN10.5 (C4), CN10.6 (C3), CN10.7 (C2), CN10.8 (C1), CN11.5 (C4), CN11.6 (C3), CN11.7 (C2), CN11.8 (C1), CN12.5 (C4), CN12.6 (C3), CN12.7 (C2), CN12.8 (C1), CN13.5 (C4), CN13.6 (C3), CN13.7 (C2), CN13.8 (C1), CN14.5 (C4), CN14.6 (C3), CN14.7 (C2), CN14.8 (C1), CN15.5 (C4), CN15.6 (C3), CN15.7 (C2), CN15.8 (C1), CN16.5 (C4), CN16.6 (C3), CN16.7 (C2), CN16.8 (C1), CN2.5 (C4), CN2.6 (C3), CN2.7 (C2), CN2.8 (C1), CN3.5 (C4), CN3.6 (C3), CN3.7 (C2), CN3.8 (C1), CN4.5 (C4), CN4.6 (C3), CN4.7 (C2), CN4.8 (C1), CN5.5 (C4), CN5.6 (C3), CN5.7 (C2), CN5.8 (C1), CN6.5 (C4), CN6.6 (C3), CN6.7 (C2), CN6.8 (C1), CN7.5 (C4), CN7.6 (C3), CN7.7 (C2), CN7.8 (C1), CN8.5 (C4), CN8.6 (C3), CN8.7 (C2), CN8.8 (C1), CN9.5 (C4), CN9.6 (C3), CN9.7 (C2), CN9.8 (C1)
- net at RN1.12 (R5.2): now also CN2.1 (common)
- net at RN1.11 (R6.2): now also CN2.2 (common)
- net at RN1.10 (R7.2): now also CN2.3 (common)
- net at RN1.9 (R8.2): now also CN2.4 (common)
- net at RN3.16 (R1.2): now also CN4.1 (common)
- net at RN3.15 (R2.2): now also CN4.2 (common)
- net at RN3.14 (R3.2): now also CN4.3 (common)
- net at RN3.13 (R4.2): now also CN4.4 (common)
- net at RN3.10 (R7.2): now also CN3.3 (common)
- net at RN3.11 (R6.2): now also CN3.2 (common)
- net at RN3.12 (R5.2): now also CN3.1 (common)
- net at RN3.9 (R8.2): now also CN3.4 (common)
- net at RN15.12 (R5.2): now also CN15.1 (common)
- net at RN15.11 (R6.2): now also CN15.2 (common)
- net at RN15.10 (R7.2): now also CN15.3 (common)
- net at RN15.9 (R8.2): now also CN15.4 (common)
- net at RN15.13 (R4.2): now also CN16.4 (common)
- net at RN15.14 (R3.2): now also CN16.3 (common)
- net at RN15.15 (R2.2): now also CN16.2 (common)
- net at RN15.16 (R1.2): now also CN16.1 (common)
- net at RN9.4 (R4.1): now also CN11.1 (common)
- net at RN9.3 (R3.1): now also CN11.2 (common)
- net at RN9.2 (R2.1): now also CN11.3 (common)
- net at RN9.1 (R1.1): now also CN11.4 (common)
- net at RN13.12 (R5.2): now also CN13.1 (common)
- net at RN13.11 (R6.2): now also CN13.2 (common)
- net at RN13.10 (R7.2): now also CN13.3 (common)
- net at RN13.9 (R8.2): now also CN13.4 (common)
- net at RN4.12 (R5.2): now also CN8.1 (common)
- net at RN4.11 (R6.2): now also CN8.2 (common)
- net at RN4.10 (R7.2): now also CN8.3 (common)
- net at RN4.9 (R8.2): now also CN8.4 (common)
- net at RN11.10 (R7.2): now also CN6.3 (common)
- net at RN11.11 (R6.2): now also CN6.2 (common)
- net at RN11.12 (R5.2): now also CN6.1 (common)
- net at RN11.13 (R4.2): now also CN5.4 (common)
- net at RN11.14 (R3.2): now also CN5.3 (common)
- net at RN11.15 (R2.2): now also CN5.2 (common)
- net at RN11.16 (R1.2): now also CN5.1 (common)
- net at RN11.9 (R8.2): now also CN6.4 (common)
- net at RN8.10 (R7.2): now also CN10.3 (common)
- net at RN8.11 (R6.2): now also CN10.2 (common)
- net at RN8.12 (R5.2): now also CN10.1 (common)
- net at RN8.13 (R4.2): now also CN9.4 (common)
- net at RN8.14 (R3.2): now also CN9.3 (common)
- net at RN8.15 (R2.2): now also CN9.2 (common)
- net at RN8.16 (R1.2): now also CN9.1 (common)
- net at RN8.9 (R8.2): now also CN10.4 (common)
- net at RN9.8 (R8.1): now also CN12.1 (common)
- net at RN9.7 (R7.1): now also CN12.2 (common)
- net at RN9.6 (R6.1): now also CN12.3 (common)
- net at RN9.5 (R5.1): now also CN12.4 (common)
- net at RN4.13 (R4.2): now also CN7.4 (common)
- net at RN4.14 (R3.2): now also CN7.3 (common)
- net at RN4.15 (R2.2): now also CN7.2 (common)
- net at RN4.16 (R1.2): now also CN7.1 (common)
- net at RN13.16 (R1.2): now also CN14.1 (common)
- net at RN13.15 (R2.2): now also CN14.2 (common)
- net at RN13.14 (R3.2): now also CN14.3 (common)
- net at RN13.13 (R4.2): now also CN14.4 (common)
Other:
- moved on the sheet: RN1, RN11, RN13, RN15, RN3, RN4, RN8, RN9
