File: boards/Zx50_Backplane_RevD/Zx50_Backplane_RevD.kicad_pcb (KiCad board)
At the start: 4 copper layers, 210.8 x 137.2 mm, 75 parts, among them CN1 100pF, CN10 100pF, CN11 100pF, CN12 100pF, CN13 100pF, CN14 100pF, CN15 100pF, CN16 100pF, CN2 100pF, CN3 100pF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

Commit message: pico async is ok, merge to master.  Also add recent work on hw boards
Parts:
- C10, C12, C13, C14: value 100pF -> 47pF; footprint Capacitor_SMD:C_0805_2012Metric_Pad1.18x1.45mm_HandSolder -> Capacitor_SMD:C_0805_2012Metric
- C2, C3, C4, C5, C6, C7, C8, C9: footprint Capacitor_SMD:C_0805_2012Metric_Pad1.18x1.45mm_HandSolder -> Capacitor_SMD:C_0805_2012Metric
- CN1, CN10, CN11, CN12, CN13, CN14, CN15, CN16, CN2, CN3, CN4, CN5, CN6, CN7, CN8, CN9: value 100pF -> 47pF
- R10, R2, R3, R8, R9: value 100 -> 100R; footprint Resistor_SMD:R_0805_2012Metric_Pad1.20x1.40mm_HandSolder -> Resistor_SMD:R_0805_2012Metric
