File: boards/Zx50_MemoryCard_RevC1/fpga_mem_RevC1.kicad_sch (KiCad schematic)
At the start: 94 parts, among them J10 RS232 5V, J8 DEBUG, J9 JTAG 5V, SW2 RESET, U12 LCMXO3LF-6900C-5BG400C, U13 TXU0204PWR, U14 TXU0304PWR, Y1 25 MHz

Commit message: reorg firmware
Parts:
- removed R42, R43: 33, Resistor_SMD:R_0402_1005Metric, symbol Device:R_Small
- added D14: RED, LED_SMD:LED_0805_2012Metric, symbol Device:LED_Small
- added D15, D16, D17, D18: BLUE, LED_SMD:LED_0805_2012Metric, symbol Device:LED_Small
- added D19, D20: GRN, LED_SMD:LED_0805_2012Metric, symbol Device:LED_Small
- R10, R11, R12, R13, R14, R8, R9: value 33 -> 330; footprint Resistor_SMD:R_0402_1005Metric -> Resistor_SMD:R_0805_2012Metric; LCSC C25076 -> C17630; MFG_PN 0402WGF1000TCE -> 0805W8F3300T5E
- R41: value 33 -> 10k; LCSC C25076 -> C25744; MFG_PN 0402WGF1000TCE -> 0402W8F1002T5E; now in the parts list
Connections:
- net ~OE is gone; now on net +3.3V: R9.2
- net ~SH_D_OE is gone; now on net +3.3V: R8.2
- net +3.3V: now also R10.2, R11.2, R12.2, R13.2, R14.2, R41.2
- net D_DIR: no longer R10.1, R41.2
- net ~Z80_D_OE: no longer R11.1
- net CE3_LED_N: now reaches R41.1
- net CE3_LED_N: now also D18.1 (K)
- net at R9.1: now also D15.2 (A)
- net at R8.1: now also D14.2 (A)
- net RAM2.A10: now reaches U12.L16 (PR16C)
- net RAM2.A19: now reaches U12.L17 (PR12D)
- net RAM2.A15: now reaches U12.L20 (PR15B)
- net RAM2.A14: now reaches U12.M15 (PR19C)
- net RAM2.A13: now reaches U12.M16 (PR17C)
- net RAM2.A12: now reaches U12.M17 (PR17A)
- net RAM2.A11: now reaches U12.M18 (PR16D)
- net RAM2.A18: now reaches U12.M19 (PR16B)
- net RAM2.A17: now reaches U12.M20 (PR16A)
- net RAM2.A6: now reaches U12.N15 (PR23C)
- net RAM2.A7: now reaches U12.N16 (PR21A)
- net RAM2.A9: now reaches U12.N17 (PR18B)
- net RAM2.A8: now reaches U12.N18 (PR18A)
- net RAM2.D7: now reaches U12.N19 (PR17D)
- net RAM2.OE_N: now reaches U12.N20 (PR17B)
- net RAM2.A2: now reaches U12.P15 (PR24C)
- net RAM2.A3: now reaches U12.P16 (PR23B)
- net RAM2.A5: now reaches U12.P17 (PR22B)
- net RAM2.A4: now reaches U12.P18 (PR19A)
- net RAM2.D5: now reaches U12.P19 (PR18D)
- net RAM2.D6: now reaches U12.P20 (PR18C)
- net RAM2.A0: now reaches U12.R16 (PR24D)
- net RAM2.A1: now reaches U12.R17 (PR24A)
- net RAM2.WE_N: now reaches U12.R19 (PR21B)
- net RAM2.D4: now reaches U12.R20 (PR19B)
- net RAM2.D2: now reaches U12.T19 (PR21D)
- net RAM2.D3: now reaches U12.T20 (PR21C)
- net RAM2.D0: now reaches U12.U19 (PR22D)
- net RAM2.D1: now reaches U12.U20 (PR22A)
- net RAM2.CE_N: now reaches U12.V20 (PR23A)
- net RAM1.A0 renamed RAM2.A16
- net ~CE0: no longer names the net of R16.1
- net ~CE0: no longer R14.1
- net ~CE1: no longer names the net of R13.1
- net ~CE1: now also D19.2 (A); no longer R17.1
- net ~CE2: no longer names the net of R18.1
- net ~WE: no longer names the net of R12.1
- net ~WE: now also D18.2 (A); no longer R15.1
- new net: D20.2 (A), R14.1
- new net: D16.2 (A), R10.1
- new net: D17.2 (A), R11.1
- new net CE0_LED_N: D15.1 (K)
- new net CE1_LED_N: D16.1 (K)
- new net CE2_LED_N: D17.1 (K)
- new net CE4_LED_N: D19.1 (K)
- new net CE5_LED_N: D20.1 (K)
- new net WE_LED_N: D14.1 (K)
Other:
- moved on the sheet: C18, C19, C20, C21, C22, C23, C24, C25, C26, C27, C28, C29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
