File: boards/Zx50_MemoryCard_RevC1/fpga_mem_RevC1.kicad_sch (KiCad schematic)
At the start: 99 parts, among them J10 RS232 5V, J8 DEBUG, J9 JTAG 5V, SW2 RESET, U12 LCMXO3LF-6900C-5BG400C, U13 TXU0204PWR, U14 TXU0304PWR, Y1 25 MHz

Commit message: updates to memory card and other changes
Parts:
- removed C19, C20, C21, C25, C26, C27, C70, C71, C72, C73: 100n, Capacitor_SMD:C_0402_1005Metric, symbol zx50_symbols:C_100n_402
- removed R15, R16, R17, R18, R41: 10k, Resistor_SMD:R_0402_1005Metric, symbol Device:R_Small
Connections:
- net CE0_LED_N: now also U12.G11 (PT25C)
- net CE1_LED_N: now also U12.G12 (PT28C)
- net CE2_LED_N: now also U12.G13 (PT33C)
- net CE3_LED_N: now also U12.R10 (PB16D)
- net CE4_LED_N: now also U12.M14 (PR19D)
- net CE5_LED_N: now also U12.N14 (PR23D)
- net DBG0: now also U12.H14 (PR4C)
- net DBG1: now also U12.H15 (PR4D)
- net DBG2: now also U12.J14 (PR7C)
- net DBG3: now also U12.J15 (PR7D)
- net DBG4: now also U12.J16 (PR10B)
- net DBG5: now also U12.K15 (PR10D)
- net DBG6: now also U12.K16 (PR12C)
- net DBG7: now also U12.L15 (PR15D)
- net DBG_CLK: now also U12.G14 (PT35C)
- net DONE: no longer U12.A10 (PT18B)
- net RAM0.A0: no longer U12.L6 (PL16C)
- net RAM1.A5: now also U12.H18 (PR9A); no longer U12.K18 (PR11D)
- net RAM1.A6: now also U12.J17 (PR9C); no longer U12.K17 (PR11C)
- net RAM1.A8: now also U12.K17 (PR11C); no longer U12.J17 (PR9C)
- net RAM1.A9: now also U12.K18 (PR11D); no longer U12.H18 (PR9A)
- net U.RX2_CLK_N: now also U12.B12 (PT22B); no longer U12.B14 (PT26B)
- net U.RX2_CLK_P: now also U12.A12 (PT22A); no longer U12.A14 (PT26A)
- net U.RX2_DAT_N: now also U12.B14 (PT26B); no longer U12.B17 (PT32B)
- net U.RX2_DAT_P: now also U12.A14 (PT26A); no longer U12.A17 (PT32A)
- net U.TX2_CLK_N: now also U12.B15 (PT27B); no longer U12.B18 (PT34B)
- net U.TX2_CLK_P: now also U12.A15 (PT27A); no longer U12.A18 (PT34A)
- net U.TX2_DAT_N: now also U12.A16 (PT28A); no longer U12.A20 (PT36B)
- net U.TX2_DAT_P: now also U12.B16 (PT28B); no longer U12.B19 (PT36A)
- net WE_LED_N: now also U12.E7 (PT11D)
- net ~LED0: now also U12.D5 (PT10D)
- net ~LED1: now also U12.D6 (PT11C)
- net ~LED2: now also U12.D7 (PT12D)
- net ~LED3: now also U12.E6 (PT10C)
- net U.~GRN2: now reaches U12.C11 (PT22C)
- net U.~YLW2: now reaches U12.D11 (PT22D)
- net RAM1.A0: now reaches U12.H16 (PR8C)
- net A_DIR: now reaches U12.P6 (PL24D)
- net CARD_A3: now reaches U12.P12 (PB29C)
- net CARD_A1: now reaches U12.P13 (PB32C)
- net ~BOOT_EN: now reaches U12.P14 (PB37C)
- net CARD_A2: now reaches U12.R12 (PB29D)
- net CARD_A0: now reaches U12.R13 (PB32D)
- net B.G14: now reaches U12.R14 (PB37D)
- net B.G15: now reaches U12.R15 (PB38D)
- net B.G11: now reaches U12.T12 (PB31C)
- net B.G12: now reaches U12.T13 (PB31D)
- net B.G13: now reaches U12.T14 (PB35C)
- net B.G2: now reaches U12.T16 (PB38C)
- net B.G1: now reaches U12.T17 (PR25B)
- net B.G0: now reaches U12.T18 (PR22C)
- net B.G8: now reaches U12.U11 (PB21C)
- net B.G9: now reaches U12.U12 (PB28C)
- net B.G10: now reaches U12.U14 (PB34B)
- net G_DIR: now reaches U12.U15 (PB35D)
- net B.G4: now reaches U12.U17 (PR25C)
- net B.G3: now reaches U12.U18 (PR24B)
- net ~SH_D_OE: now reaches U12.V12 (PB26C)
- net B.~BUSRQ: now reaches U12.V13 (PB26D)
- net B.~WAIT: now reaches U12.V14 (PB34A)
- net B.~INT: now reaches U12.V15 (PB34C)
- net B.G7: now reaches U12.V16 (PB34D)
- net B.G6: now reaches U12.V17 (PR25D)
- net B.G5: now reaches U12.V19 (PR25A)
- net SH_D_DIR: now reaches U12.W11 (PB21B)
- net SH_C_DIR: now reaches U12.W12 (PB23B)
- net B.~SH_STB: now reaches U12.W13 (PB26B)
- net B.~SH_EN: now reaches U12.W14 (PB28B)
- net B.~SH_DONE: now reaches U12.W15 (PB29B)
- net B.SD1: now reaches U12.W16 (PB31B)
- net B.SD3: now reaches U12.W17 (PB32B)
- net B.SD5: now reaches U12.W18 (PB35B)
- net B.SD7: now reaches U12.W19 (PB37B)
- net G_OE_N: now reaches U12.W20 (PB38B)
- net B.~SH_BUSY: now reaches U12.Y11 (PB21A)
- net ~SH_C_OE: now reaches U12.Y13 (PB26A)
- net B.~SH_INC: now reaches U12.Y14 (PB28A)
- net B.SH_RW: now reaches U12.Y15 (PB29A)
- net B.SD0: now reaches U12.Y16 (PB31A)
- net B.SD2: now reaches U12.Y17 (PB32A)
- net B.SD4: now reaches U12.Y18 (PB35A)
- net B.SD6: now reaches U12.Y19 (PB37A)
- net D_DIR renamed Z80_D_DIR
- new net UROM1.CE_N: U12.B19 (PT36A)
- new net UROM1.HOLD_N: U12.A20 (PT36B)
- new net UROM1.SCK: U12.A17 (PT32A)
- new net UROM1.SI: U12.B17 (PT32B)
- new net UROM1.SO: U12.B18 (PT34B)
- new net UROM1.WP_N: U12.A18 (PT34A)
- no-connect marks 23 -> 70
Other:
- moved on the sheet: C74, C75, C77
