File: boards/Zx50_MemoryCard_RevC1/Zx50_MemoryCard_RevC1.kicad_pcb (KiCad board)
At the start: 6 copper layers, 132.1 x 107.9 mm, 254 parts, among them J1 2.5V, J10 RS232 5V, J11 RJ45_RB1-125B8G1A, J12 RJ45_RB1-125B8G1A, J2 3.3V, J3 Zx50_EdgeConnector, J4 TP_CLK, J5 TP_MCLK, J6 GND, J7 GND, J8 DEBUG, J9 JTAG 5V, Q1 2N7002, SW1 SW_DIP_x05, SW2 RESET, U1 AMS1117-2.5, U10 74LVC3G07, U11 74LVC245, U12 LCMXO3LF-6900C-5BG400C, U13 TXU0204PWR, U14 TXU0304PWR, U15 IS61WV10248EDBLL, U16 IS61WV10248EDBLL, U17 IS61WV10248EDBLL, U18 IS61WV10248EDBLL, U19 IS25LP080D-JNLE-TR, U2 AMS1117-3.3, U20 IS25LP080D-JNLE-TR, U21 74LVC245, U22 SN74LVC1G17DBVR, U23 74LVC245, U24 74LVC245, U3 74LVC245, U4 74LVC245, U5 74LVC245, U6 74LVC245, U7 74LVC1G17, U8 74LVC1G17, U9 74LVC245, Y1 25 MHz

Commit message: updates to memory card and other changes
Parts:
- removed C19, C20, C21, C25, C26, C27, C70, C71, C72, C73: 100n, Capacitor_SMD:C_0402_1005Metric
- removed the C60 at (213.9, 143.2)
- removed the C62 at (229.1, 155.2)
- removed the C63 at (229.1, 160.0)
- removed Q1: 2N7002, digikey-footprints:SOT-23-3
- removed R15, R16, R17, R18, R41: 10k, Resistor_SMD:R_0402_1005Metric
- removed R42, R43: 33, Resistor_SMD:R_0402_1005Metric
- removed R77: 10k, Resistor_SMD:R_0805_2012Metric
- added RN2: 33R, Resistor_SMD:R_Array_Convex_8x0602, F.Cu at (109.8, 155.3)
- added RN3: 33R, Resistor_SMD:R_Array_Convex_8x0602, F.Cu at (118.7, 155.3)
- added RN4: 33R, Resistor_SMD:R_Array_Convex_8x0602, F.Cu at (61.8, 137.1)
- R1, R113, R118, R119, R2, R32, R40, R68, R73, R76: moved to B.Cu
- moved R1 203.1 mm to (59.6, 127.5), turned to 90 degrees
- moved C40 179.3 mm to (52.3, 77.7), turned to 180 degrees
- moved R23 179.0 mm to (52.3, 76.4)
- moved R40 142.1 mm to (96.2, 109.5)
- moved C83 134.3 mm to (125.8, 135.8), turned to -90 degrees
- moved R32 127.2 mm to (108.4, 92.7), turned to 90 degrees
- moved R124 126.9 mm to (115.6, 95.5)
- moved R120 125.8 mm to (118.2, 85.7), turned to -90 degrees
- moved R99 125.4 mm to (114.6, 91.7)
- moved R76 124.7 mm to (111.7, 148.8), turned to 180 degrees
- moved R125 123.9 mm to (123.4, 92.0)
- moved R73 123.6 mm to (107.9, 149.6)
- moved R98 123.4 mm to (114.6, 93.0)
- moved R97 121.4 mm to (114.6, 94.2)
- moved R101 121.0 mm to (114.5, 89.0)
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Connections:
- C16 pad 1: +5V -> +3.3V
- C54 pad 1: /FPGA/RDMA/RDMA_CT -> /FPGA/RDMA/RDMA_CT1
- C55 pad 1: /FPGA/RDMA/RDMA_CT -> /FPGA/RDMA/RDMA_CT2
- J11 pad 1: /FPGA/RDMA/RDMA_CT -> /FPGA/RDMA/RDMA_CT1
- J12 pad 1: /FPGA/RDMA/RDMA_CT -> /FPGA/RDMA/RDMA_CT2
- R120 pad 1: /FPGA/memory/ROM1.HOLD_N -> +2V5
- R120 pad 2: +2V5 -> /FPGA/UROM1.HOLD_N
- R3 pad 1: GND -> /~SH_C_OE
- R73 pad 2: Net-(U9-A6) -> Net-(RN2-R7.2)
- R76 pad 2: Net-(U9-B6) -> Net-(U9-B7)
- RN1 pad 6: Net-(RN1-R5) -> /CARD_A3
- SW1 pad 5: Net-(RN1-R5) -> /CARD_A3
- U10 pad 8: +5V -> +3.3V
- U11 pad 1: /D_DIR -> /SH_D_DIR
- U11 pad 11: /B.D7 -> /B.SD7
- U11 pad 12: /B.D6 -> /B.SD6
- U11 pad 13: /B.D5 -> /B.SD5
- U11 pad 14: /B.D4 -> /B.SD4
- U11 pad 15: /B.D3 -> /B.SD3
- U11 pad 16: /B.D2 -> /B.SD2
- U11 pad 17: /B.D1 -> /B.SD1
- U11 pad 18: /B.D0 -> /B.SD0
- U11 pad 2: /SD0 -> Net-(RN3-R1.2)
- U11 pad 3: /SD1 -> Net-(RN3-R2.2)
- U11 pad 4: /SD2 -> Net-(RN3-R3.2)
- U11 pad 5: /SD3 -> Net-(RN3-R4.2)
- U11 pad 6: /SD4 -> Net-(RN3-R5.2)
- U11 pad 7: /SD5 -> Net-(RN3-R6.2)
- U11 pad 8: /SD6 -> Net-(RN3-R7.2)
- U11 pad 9: /SD7 -> Net-(RN3-R8.2)
- U12 pad A10: /FPGA/DONE -> unconnected-(U12B-PT18B-PadA10)
- U12 pad A12: unconnected-(U12B-PT22A-PadA12) -> /FPGA/U.RX2_CLK_P
- U12 pad A14: /FPGA/U.RX2_CLK_P -> /FPGA/U.RX2_DAT_P
- U12 pad A15: unconnected-(U12B-PT27A-PadA15) -> /FPGA/U.TX2_CLK_P
- U12 pad A16: unconnected-(U12B-PT28A-PadA16) -> /FPGA/U.TX2_DAT_N
- U12 pad A17: /FPGA/U.RX2_DAT_P -> /FPGA/UROM1.SCK
- U12 pad A18: /FPGA/U.TX2_CLK_P -> /FPGA/UROM1.WP_N
- U12 pad A20: /FPGA/U.TX2_DAT_N -> /FPGA/UROM1.HOLD_N
- U12 pad B12: unconnected-(U12B-PT22B-PadB12) -> /FPGA/U.RX2_CLK_N
- U12 pad B14: /FPGA/U.RX2_CLK_N -> /FPGA/U.RX2_DAT_N
- U12 pad B15: unconnected-(U12B-PT27B-PadB15) -> /FPGA/U.TX2_CLK_N
- U12 pad B16: unconnected-(U12B-PT28B-PadB16) -> /FPGA/U.TX2_DAT_P
- U12 pad B17: /FPGA/U.RX2_DAT_N -> /FPGA/UROM1.SI
- U12 pad B18: /FPGA/U.TX2_CLK_N -> /FPGA/UROM1.SO
- U12 pad B19: /FPGA/U.TX2_DAT_P -> /FPGA/UROM1.CE_N
- U12 pad C11: unconnected-(U12C-PT22C-PadC11) -> /FPGA/U.~GRN2
- U12 pad D11: unconnected-(U12C-PT22D-PadD11) -> /FPGA/U.~YLW2
- U12 pad D5: unconnected-(U12A-PT10D-PadD5) -> /FPGA/~LED0
- U12 pad D6: unconnected-(U12A-PT11C-PadD6) -> /FPGA/~LED1
- U12 pad D7: unconnected-(U12A-PT12D-PadD7) -> /FPGA/~LED2
- U12 pad E6: unconnected-(U12A-PT10C-PadE6) -> /FPGA/~LED3
- U12 pad E7: unconnected-(U12A-PT11D-PadE7) -> /FPGA/WE_LED_N
- U12 pad G11: unconnected-(U12C-PT25C-PadG11) -> /FPGA/CE0_LED_N
- U12 pad G12: unconnected-(U12C-PT28C-PadG12) -> /FPGA/CE1_LED_N
- U12 pad G13: unconnected-(U12C-PT33C-PadG13) -> /FPGA/CE2_LED_N
- U12 pad G14: unconnected-(U12C-PT35C-PadG14) -> /FPGA/DBG_CLK
- U12 pad H14: unconnected-(U12C-PR4C-PadH14) -> /FPGA/DBG0
- U12 pad H15: unconnected-(U12C-PR4D-PadH15) -> /FPGA/DBG1
- U12 pad H16: unconnected-(U12C-PR8C-PadH16) -> /FPGA/RAM1.A0
- U12 pad H18: /FPGA/RAM1.A9 -> /FPGA/RAM1.A5
- U12 pad J14: unconnected-(U12C-PR7C-PadJ14) -> /FPGA/DBG2
- U12 pad J15: unconnected-(U12C-PR7D-PadJ15) -> /FPGA/DBG3
- U12 pad J16: unconnected-(U12C-PR10B-PadJ16) -> /FPGA/DBG4
- U12 pad J17: /FPGA/RAM1.A8 -> /FPGA/RAM1.A6
- U12 pad K15: unconnected-(U12C-PR10D-PadK15) -> /FPGA/DBG5
- U12 pad K16: unconnected-(U12C-PR12C-PadK16) -> /FPGA/DBG6
- U12 pad K17: /FPGA/RAM1.A6 -> /FPGA/RAM1.A8
- U12 pad K18: /FPGA/RAM1.A5 -> /FPGA/RAM1.A9
- U12 pad L15: unconnected-(U12C-PR15D-PadL15) -> /FPGA/DBG7
- U12 pad L6: /FPGA/RAM0.A0 -> unconnected-(U12A-PL16C-PadL6)
- U12 pad M14: unconnected-(U12D-PR19D-PadM14) -> /FPGA/CE4_LED_N
- U12 pad N14: unconnected-(U12D-PR23D-PadN14) -> /FPGA/CE5_LED_N
- U12 pad P12: unconnected-(U12D-PB29C-PadP12) -> /CARD_A3
- U12 pad P13: unconnected-(U12D-PB32C-PadP13) -> /CARD_A1
- U12 pad P14: unconnected-(U12D-PB37C-PadP14) -> /~BOOT_EN
- U12 pad P6: unconnected-(U12B-PL24D-PadP6) -> /A_DIR
- U12 pad R10: unconnected-(U12D-PB16D-PadR10) -> /FPGA/CE3_LED_N
- U12 pad R12: unconnected-(U12D-PB29D-PadR12) -> /CARD_A2
- U12 pad R13: unconnected-(U12D-PB32D-PadR13) -> /CARD_A0
- U12 pad R14: unconnected-(U12D-PB37D-PadR14) -> /B.G14
- U12 pad R15: unconnected-(U12D-PB38D-PadR15) -> /B.G15
- U12 pad T12: unconnected-(U12D-PB31C-PadT12) -> /B.G11
- U12 pad T13: unconnected-(U12D-PB31D-PadT13) -> /B.G12
- U12 pad T14: unconnected-(U12D-PB35C-PadT14) -> /B.G13
- U12 pad T16: unconnected-(U12D-PB38C-PadT16) -> /B.G2
- U12 pad T17: unconnected-(U12D-PR25B-PadT17) -> /B.G1
- U12 pad T18: unconnected-(U12D-PR22C-PadT18) -> /B.G0
- U12 pad U11: unconnected-(U12D-PB21C-PadU11) -> /B.G8
- U12 pad U12: unconnected-(U12D-PB28C-PadU12) -> /B.G9
- U12 pad U14: unconnected-(U12D-PB34B-PadU14) -> /B.G10
- U12 pad U15: unconnected-(U12D-PB35D-PadU15) -> /G_DIR
- U12 pad U17: unconnected-(U12D-PR25C-PadU17) -> /B.G4
- U12 pad U18: unconnected-(U12D-PR24B-PadU18) -> /B.G3
- U12 pad V12: unconnected-(U12D-PB26C-PadV12) -> /~SH_D_OE
- U12 pad V13: unconnected-(U12D-PB26D-PadV13) -> /B.~BUSRQ
- U12 pad V14: unconnected-(U12D-PB34A-PadV14) -> /B.~WAIT
- U12 pad V15: unconnected-(U12D-PB34C-PadV15) -> /B.~INT
- U12 pad V16: unconnected-(U12D-PB34D-PadV16) -> /B.G7
- U12 pad V17: unconnected-(U12D-PR25D-PadV17) -> /B.G6
- U12 pad V19: unconnected-(U12D-PR25A-PadV19) -> /B.G5
- U12 pad V6: /D_DIR -> /Z80_D_DIR
- U12 pad W11: unconnected-(U12D-PB21B-PadW11) -> /SH_D_DIR
- U12 pad W12: unconnected-(U12D-PB23B-PadW12) -> /SH_C_DIR
- U12 pad W13: unconnected-(U12D-PB26B-PadW13) -> /B.~SH_STB
- U12 pad W14: unconnected-(U12D-PB28B-PadW14) -> /B.~SH_EN
- U12 pad W15: unconnected-(U12D-PB29B-PadW15) -> /B.~SH_DONE
- U12 pad W16: unconnected-(U12D-PB31B-PadW16) -> /B.SD1
- U12 pad W17: unconnected-(U12D-PB32B-PadW17) -> /B.SD3
- U12 pad W18: unconnected-(U12D-PB35B-PadW18) -> /B.SD5
- U12 pad W19: unconnected-(U12D-PB37B-PadW19) -> /B.SD7
- U12 pad W20: unconnected-(U12D-PB38B-PadW20) -> /G_OE_N
- U12 pad Y11: unconnected-(U12D-PB21A-PadY11) -> /B.~SH_BUSY
- U12 pad Y13: unconnected-(U12D-PB26A-PadY13) -> /~SH_C_OE
- U12 pad Y14: unconnected-(U12D-PB28A-PadY14) -> /B.~SH_INC
- U12 pad Y15: unconnected-(U12D-PB29A-PadY15) -> /B.SH_RW
- U12 pad Y16: unconnected-(U12D-PB31A-PadY16) -> /B.SD0
- U12 pad Y17: unconnected-(U12D-PB32A-PadY17) -> /B.SD2
- U12 pad Y18: unconnected-(U12D-PB35A-PadY18) -> /B.SD4
- U12 pad Y19: unconnected-(U12D-PB37A-PadY19) -> /B.SD6
- U20 pad 7: /FPGA/memory/ROM1.HOLD_N -> /FPGA/UROM1.HOLD_N
- U23 pad 1: /G_GIR -> /G_DIR
- U23 pad 11: /B.G7 -> /B.G0
- U23 pad 12: /B.G6 -> /B.G1
- U23 pad 13: /B.G5 -> /B.G2
- U23 pad 14: /B.G4 -> /B.G3
- U23 pad 15: /B.G3 -> /B.G4
- U23 pad 16: /B.G2 -> /B.G5
- U23 pad 17: /B.G1 -> /B.G6
- U23 pad 18: /B.G0 -> /B.G7
- U23 pad 2: /G0 -> /G7
- U23 pad 3: /G1 -> /G6
- U23 pad 4: /G2 -> /G5
- U23 pad 5: /G3 -> /G4
- U23 pad 6: /G4 -> /G3
- U23 pad 7: /G5 -> /G2
- U23 pad 8: /G6 -> /G1
- U23 pad 9: /G7 -> /G0
- U24 pad 1: /G_GIR -> /G_DIR
- U5 pad 1: /D_DIR -> /Z80_D_DIR
- U5 pad 2: /D0 -> Net-(RN4-R1.2)
- U5 pad 3: /D1 -> Net-(RN4-R2.2)
- U5 pad 4: /D2 -> Net-(RN4-R3.2)
- U5 pad 5: /D3 -> Net-(RN4-R4.2)
- U5 pad 6: /D4 -> Net-(RN4-R5.2)
- U5 pad 7: /D5 -> Net-(RN4-R6.2)
- U5 pad 8: /D6 -> Net-(RN4-R7.2)
- U5 pad 9: /D7 -> Net-(RN4-R8.2)
- U9 pad 1: GND -> /SH_C_DIR
- U9 pad 11: Net-(U9-B6) -> Net-(U9-B7)
- U9 pad 12: Net-(U9-B6) -> Net-(U9-B7)
- U9 pad 13: Net-(U9-B6) -> Net-(RN2-R6.2)
- U9 pad 14: GND -> /B.~SH_DONE
- U9 pad 15: GND -> /B.SH_RW
- U9 pad 16: GND -> /B.~SH_EN
- U9 pad 17: GND -> /B.~SH_INC
- U9 pad 18: GND -> /B.~SH_STB
- U9 pad 19: GND -> /~SH_C_OE
- U9 pad 2: /~SH_STB -> Net-(RN2-R1.2)
- U9 pad 3: /~SH_INC -> Net-(RN2-R2.2)
- U9 pad 4: /~SH_EN -> Net-(RN2-R3.2)
- U9 pad 5: /SH_RW -> Net-(RN2-R4.2)
- U9 pad 6: /~SH_DONE -> Net-(RN2-R5.2)
- U9 pad 7: Net-(U9-A6) -> /B.~SH_BUSY
- U9 pad 8: Net-(U9-A6) -> Net-(RN2-R7.2)
- U9 pad 9: Net-(U9-A6) -> Net-(RN2-R7.2)
Routing:
- net /FPGA/CE5_LED_N: track 2.21 -> 157.6 mm, vias 1 -> 2
- net /FPGA/CE3_LED_N: track 2.21 -> 129.4 mm, vias 1 -> 2
- net /FPGA/CE2_LED_N: track 2.21 -> 126.3 mm, vias 1 -> 2
- net /FPGA/CE0_LED_N: track 2.62 -> 120.3 mm, vias 1 -> 2
- net /FPGA/CE1_LED_N: track 2.21 -> 118.7 mm, vias 1 -> 2
- net /FPGA/~LED2: track 2.21 -> 115.4 mm, vias 1 -> 3
- net /FPGA/~LED3: track 2.21 -> 115.0 mm, vias 1 -> 2
- net /FPGA/~LED1: track 2.21 -> 114.5 mm, vias 1 -> 2
- net /FPGA/WE_LED_N: track 2.21 -> 114.1 mm, vias 1 -> 2
- net /FPGA/~LED0: track 2.21 -> 112.3 mm, vias 1 -> 2
- net /FPGA/CE4_LED_N: track 2.21 -> 82.0 mm, vias 1 -> 2
- net /CARD_A3: track 0.00 -> 74.4 mm, vias 0 -> 1
- net /FPGA/INIT_N: track 0.00 -> 72.9 mm, vias 0 -> 3
- net /FPGA/DBG_CLK: track 0.00 -> 71.7 mm, vias 0 -> 1
- net /FPGA/DONE: track 0.00 -> 71.4 mm, vias 0 -> 2
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