File: boards/Zx50_MemoryCard_RevC1/Zx50_MemoryCard_RevC1.kicad_pcb (KiCad board)
At the start: 6 copper layers, 132.1 x 107.9 mm, 235 parts, among them J1 2.5V, J10 RS232 5V, J11 RJ45_RB1-125B8G1A, J12 RJ45_RB1-125B8G1A, J2 3.3V, J3 Zx50_EdgeConnector, J4 TP_CLK, J5 TP_MCLK, J6 GND, J7 GND, J8 DEBUG, J9 JTAG 5V, SW1 SW_DIP_x05, SW2 RESET, U1 AMS1117-2.5, U10 74LVC3G07, U11 74LVC245, U12 LCMXO3LF-6900C-5BG400C, U13 TXU0204PWR, U14 TXU0304PWR, U15 IS61WV10248EDBLL, U16 IS61WV10248EDBLL, U17 IS61WV10248EDBLL, U18 IS61WV10248EDBLL, U19 IS25LP080D-JNLE-TR, U2 AMS1117-3.3, U20 IS25LP080D-JNLE-TR, U21 74LVC245, U22 SN74LVC1G17DBVR, U23 74LVC245, U24 74LVC245, U3 74LVC245, U4 74LVC245, U5 74LVC245, U6 74LVC245, U7 74LVC1G17, U8 74LVC1G17, U9 74LVC245, Y1 25 MHz

Commit message: cpu revc1
Routing:
- net /FPGA/RAM3.A4: track 25.5 -> 27.4 mm
- net /FPGA/RAM3.A3: track 25.7 -> 27.7 mm
- net /FPGA/RAM3.A2: track 27.9 -> 29.8 mm
- net /FPGA/RAM3.WE_N: track 17.3 -> 18.1 mm
- net /FPGA/RAM3.CE_N: track 26.4 -> 27.1 mm
