File: boards/Zx50_MemoryCard_RevC1/Zx50_MemoryCard_RevC1.kicad_sch (KiCad schematic)
At the start: 49 parts, among them J3 Zx50_EdgeConnector, J4 TP_CLK, J5 TP_MCLK, Q1 2N7002, SW1 SW_DIP_x05, U10 74LVC3G07, U11 74LVC245, U21 74LVC245, U22 SN74LVC1G17DBVR, U23 74LVC245, U24 74LVC245, U3 74LVC245, U4 74LVC245, U5 74LVC245, U6 74LVC245, U7 74LVC1G17, U8 74LVC1G17, U9 74LVC245

Commit message: updates to memory card and other changes
Parts:
- removed Q1: 2N7002, digikey-footprints:SOT-23-3, symbol dk_Transistors-FETs-MOSFETs-Single:2N7002
- removed R77: 10k, Resistor_SMD:R_0805_2012Metric, symbol Device:R_Small
- added RN2, RN3, RN4: 33R, Resistor_SMD:R_Array_Convex_8x0602, symbol Device:R_Pack08
Connections:
- net +3.3V: now also C16.1, U10.8 (VCC)
- net +5V: no longer C16.1, U10.8 (VCC)
- net B.D0: no longer U11.18 (B1)
- net B.D1: no longer U11.17 (B2)
- net B.D2: no longer U11.16 (B3)
- net B.D3: no longer U11.15 (B4)
- net B.D4: no longer U11.14 (B5)
- net B.D5: no longer U11.13 (B6)
- net B.D6: no longer U11.12 (B7)
- net B.D7: no longer U11.11 (B8)
- net B.G0: now also U23.11 (B8); no longer U23.18 (B1)
- net B.G1: now also U23.12 (B7); no longer U23.17 (B2)
- net B.G2: now also U23.13 (B6); no longer U23.16 (B3)
- net B.G3: now also U23.14 (B5); no longer U23.15 (B4)
- net B.G4: now also U23.15 (B4); no longer U23.14 (B5)
- net B.G5: now also U23.16 (B3); no longer U23.13 (B6)
- net B.G6: now also U23.17 (B2); no longer U23.12 (B7)
- net B.G7: now also U23.18 (B1); no longer U23.11 (B8)
- net B.~SH_BUSY: now also U9.7 (A6)
- net D0: now also RN4.1 (R1.1); no longer U5.2 (A1)
- net D1: now also RN4.2 (R2.1); no longer U5.3 (A2)
- net D2: now also RN4.3 (R3.1); no longer U5.4 (A3)
- net D3: now also RN4.4 (R4.1); no longer U5.5 (A4)
- net D4: now also RN4.5 (R5.1); no longer U5.6 (A5)
- net D5: now also RN4.6 (R6.1); no longer U5.7 (A6)
- net D6: now also RN4.7 (R7.1); no longer U5.8 (A7)
- net D7: now also RN4.8 (R8.1); no longer U5.9 (A8)
- net G0: now also U23.9 (A8); no longer U23.2 (A1)
- net G1: now also U23.8 (A7); no longer U23.3 (A2)
- net G2: now also U23.7 (A6); no longer U23.4 (A3)
- net G3: now also U23.6 (A5); no longer U23.5 (A4)
- net G4: now also U23.5 (A4); no longer U23.6 (A5)
- net G5: now also U23.4 (A3); no longer U23.7 (A6)
- net G6: now also U23.3 (A2); no longer U23.8 (A7)
- net G7: now also U23.2 (A1); no longer U23.9 (A8)
- net SD0: now also RN3.1 (R1.1); no longer U11.2 (A1)
- net SD1: now also RN3.2 (R2.1); no longer U11.3 (A2)
- net SD2: now also RN3.3 (R3.1); no longer U11.4 (A3)
- net SD3: now also RN3.4 (R4.1); no longer U11.5 (A4)
- net SD4: now also RN3.5 (R5.1); no longer U11.6 (A5)
- net SD5: now also RN3.6 (R6.1); no longer U11.7 (A6)
- net SD6: now also RN3.7 (R7.1); no longer U11.8 (A7)
- net SD7: now also RN3.8 (R8.1); no longer U11.9 (A8)
- net SH_RW: now also RN2.4 (R4.1); no longer U9.5 (A4)
- net ~SH_BUSY: now also RN2.6 (R6.1)
- net ~SH_DONE: now also RN2.5 (R5.1); no longer U9.6 (A5)
- net ~SH_EN: now also RN2.3 (R3.1); no longer U9.4 (A3)
- net ~SH_INC: now also RN2.2 (R2.1); no longer U9.3 (A2)
- net ~SH_STB: now also RN2.1 (R1.1); no longer U9.2 (A1)
- net at R73.2, U9.8 (A7), U9.9 (A8): now also RN2.10 (R7.2), RN2.9 (R8.2); no longer U9.7 (A6)
- net at R76.2, U9.11 (B8), U9.12 (B7): no longer U9.13 (B6)
- net CARD_A3: now reaches RN1.6 (R5), SW1.5
- net D_DIR renamed SH_D_DIR
- net SH_D_DIR: no longer U5.1 (DIR)
- net G_GIR renamed G_DIR
- new net: RN3.10 (R7.2), U11.8 (A7)
- new net: RN3.11 (R6.2), U11.7 (A6)
- new net: RN3.12 (R5.2), U11.6 (A5)
- new net: RN3.13 (R4.2), U11.5 (A4)
- new net: RN3.14 (R3.2), U11.4 (A3)
- new net: RN3.15 (R2.2), U11.3 (A2)
- new net: RN3.16 (R1.2), U11.2 (A1)
- new net: RN3.9 (R8.2), U11.9 (A8)
- new net: RN2.11 (R6.2), U9.13 (B6)
- new net: RN2.12 (R5.2), U9.6 (A5)
- new net: RN2.13 (R4.2), U9.5 (A4)
- new net: RN2.14 (R3.2), U9.4 (A3)
- new net: RN2.15 (R2.2), U9.3 (A2)
- new net: RN2.16 (R1.2), U9.2 (A1)
- new net: RN4.16 (R1.2), U5.2 (A1)
- new net: RN4.15 (R2.2), U5.3 (A2)
- new net: RN4.14 (R3.2), U5.4 (A3)
- new net: RN4.13 (R4.2), U5.5 (A4)
- new net: RN4.12 (R5.2), U5.6 (A5)
- new net: RN4.11 (R6.2), U5.7 (A6)
- new net: RN4.10 (R7.2), U5.8 (A7)
- new net: RN4.9 (R8.2), U5.9 (A8)
- new net B.SD0: U11.18 (B1)
- new net B.SD1: U11.17 (B2)
- new net B.SD2: U11.16 (B3)
- new net B.SD3: U11.15 (B4)
- new net B.SD4: U11.14 (B5)
- new net B.SD5: U11.13 (B6)
- new net B.SD6: U11.12 (B7)
- new net B.SD7: U11.11 (B8)
- new net Z80_D_DIR: U5.1 (DIR)
- no-connect marks 4 -> 6
Other:
- sheet FPGA ports: added B{SH_D}; removed none
- note removed: "Backplane has SH_BUSY_N +5V pullup"
- moved on the sheet: C83, C84, R73, R76, U23, U24
