File: boards/Zx50_MemoryCard_RevC1/memory.kicad_sch (KiCad schematic)
At the start: 45 parts, among them U15 IS61WV10248EDBLL, U16 IS61WV10248EDBLL, U17 IS61WV10248EDBLL, U18 IS61WV10248EDBLL, U19 IS25LP080D-JNLE-TR, U20 IS25LP080D-JNLE-TR

Commit message: updates to memory card and other changes
Parts:
- removed NT10: NetTie_2, symbol Device:NetTie_2
Connections:
- net +2V5: now also R120.1; no longer R120.2
- net UROM1.HOLD_N: now also R120.2, U20.7 (~{HOLD}/~{RESET}(IO3))
- removed net ROM1.HOLD_N: R120.1, U20.7 (~{HOLD}/~{RESET}(IO3))
Other:
- moved on the sheet: R120
