File: boards/Zx50_MemoryCard_RevC1/rdma.kicad_sch (KiCad schematic)
At the start: 40 parts, among them J11 RJ45_RB1-125B8G1A, J12 RJ45_RB1-125B8G1A

Commit message: updates to memory card and other changes
Connections:
- net RDMA_CT renamed RDMA_CT1
- net RDMA_CT1: no longer C55.1, J12.1 (CT)
- new net RDMA_CT2: C55.1, J12.1 (CT)
Changed lines of the file:
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@@
 		)
 	)
-	(label "RDMA_CT"
+	(label "RDMA_CT1"
 		(at 222.25 57.15 180)
 		(effects
@@
 		)
 	)
-	(label "RDMA_CT"
+	(label "RDMA_CT2"
 		(at 222.25 132.08 180)
 		(effects
