File: boards/Zx50_Serial_RevB/Zx50_Serial.kicad_pcb (KiCad board)
At the start: 4 copper layers, 132.1 x 81.9 mm, 25 parts, among them IC1 Z80CTC, IC2 Z80DART, J1 Zx50_EdgeConnector, J2 DE9_Socket, J3 DB9-USB-D5-F, J4 PortA, J5 PortB, U1 74AHCT138, U4 MAX232ACPE, Y1 7.3728 MHz

Commit message: ctc_tick.z80 working, CPU RevB done
Parts:
- Y1: value 7.3728 MHz -> 1.8432 MHz
Connections:
- IC1 pad 20: unconnected-(IC1-TRG3-Pad20) -> Net-(IC1-TO2)
- IC1 pad 21: unconnected-(IC1-TRG2-Pad21) -> /OSC
- IC1 pad 9: unconnected-(IC1-TO2-Pad9) -> Net-(IC1-TO2)
Routing:
- net Net-(IC1-TO2): track 0.00 -> 15.2 mm
- net /OSC: track 9.53 -> 12.1 mm
Other:
- board text added: "Zx50 Serial I/O Marc Mosko, 2026 Zx50_Serial_RevB1"
- board text removed: "Zx50 Serial I/O Marc Mosko, 2026 Zx50_Serial_RevB"
