File: boards/Zx50_Serial_RevB/Zx50_Serial.kicad_sch (KiCad schematic)
At the start: 24 parts, among them IC1 Z80CTC, IC2 Z80DART, J1 Zx50_EdgeConnector, J2 DE9_Socket, J3 DB9-USB-D5-F, J4 PortA, J5 PortB, U1 74AHCT138, U4 MAX232ACPE, Y1 7.3728 MHz

Commit message: ctc_tick.z80 working, CPU RevB done
Parts:
- Y1: value 7.3728 MHz -> 1.8432 MHz; DigiKey_PN 110-MXO45HS-3C-7M372800-ND -> (none); Mouser_PN (none) -> 520-TCH184-X; SKU MXO45HS-3C-7M372800 -> ECS-2100AX-1.8432MHZ
Connections:
- net OSC: now also IC1.21 (TRG2)
- net at IC1.20 (TRG3): now also IC1.9 (TO2)
- no-connect marks 74 -> 71
Changed lines of the file:
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@@
 	)
 	(junction
+		(at 38.1 67.31)
+		(diameter 0)
+		(color 0 0 0 0)
+	)
+	(junction
 		(at 191.77 54.61)
 		(diameter 0)
@@
 	)
 	(no_connect
-		(at 45.72 72.39)
-	)
-	(no_connect
 		(at 88.9 185.42)
 	)
@@
 	)
 	(no_connect
-		(at 53.34 72.39)
-	)
-	(no_connect
 		(at 111.76 185.42)
 	)
@@
 	)
 	(no_connect
-		(at 48.26 72.39)
-	)
-	(no_connect
 		(at 86.36 185.42)
 	)
@@
 		)
 	)
+	(wire
+		(pts
+			(xy 48.26 72.39) (xy 53.34 72.39)
+		)
+		(stroke
+			(width 0)
+			(type default)
+		)
+	)
 	(bus
 		(pts
@@
 	(wire
 		(pts
+			(xy 45.72 72.39) (xy 45.72 67.31)
+		)
+		(stroke
+			(width 0)
+			(type default)
+		)
+	)
+	(wire
+		(pts
 			(xy 196.85 30.48) (xy 196.85 50.8)
 		)
@@
 	(wire
 		(pts
+			(xy 45.72 67.31) (xy 38.1 67.31)
+		)
+		(stroke
+			(width 0)
+			(type default)
+		)
+	)
+	(wire
+		(pts
 			(xy 196.85 50.8) (xy 199.39 50.8)
 		)
@@
 			)
 		)
-		(property "Value" "7.3728 MHz"
+		(property "Value" "1.8432 MHz"
 			(at 34.798 48.26 90)
 			(effects
@@
 			)
 		)
-		(property "Datasheet" "https://support.epson.biz/td/api/doc_check.php?mode=dl&lang=en&Parts=SG-8002DC"
+		(property "Datasheet" ""
 			(at 24.13 53.34 0)
 			(effects
@@
 			)
 		)
-		(property "Description" "XTAL OSC XO 7.3728MHZ HCMOS TH"
+		(property "Description" "Standard Clock Oscillators DIP-8 5V 1.8432MHz"
 			(at 24.13 55.88 0)
 			(effects
@@
 			)
 		)
-		(property "DigiKey_PN" "110-MXO45HS-3C-7M372800-ND"
+		(property "DigiKey_PN" ""
 			(at 24.13 55.88 0)
 			(effects
@@
 			)
 		)
-		(property "SKU" "MXO45HS-3C-7M372800"
+		(property "SKU" "ECS-2100AX-1.8432MHZ"
+			(at 24.13 55.88 90)
+			(effects
+				(font
+					(size 1.27 1.27)
+				)
+				(hide yes)
+			)
+		)
+		(property "Mouser_PN" "520-TCH184-X"
 			(at 24.13 55.88 90)
 			(effects
