File: boards/Zx50_Cpu_RevB1/Zx50_Cpu_RevB1.kicad_pcb (KiCad board)
At the start: 4 copper layers, 133.5 x 100.3 mm, 39 parts, among them J1 Zx50_EdgeConnector, J2 FrontPanelConnect, J3 Clock Mezzanine, J4 Front Panel, J5 TP_D_DIR, J6 TP_BUSAK, Q1 BSS84, Q2 2N7002-7-F, SW1 RESET, U1 74AHC1G14, U10 74AHC1G08, U2 SN74ABT245BN, U3 SN74ABT245BN, U4 Z84C00xxP, U5 SN74ABT245BN, U6 MCP1316MT-46LE/OT, U7 SN74ABT245BN, U8 74LVC1G3208, U9 SN74AHCT74DRG4

Commit message: cpu revc1
Parts:
- added C12: 0.1uF, Capacitor_SMD:C_0805_2012Metric_Pad1.18x1.45mm_HandSolder, F.Cu at (39.4, 95.2)
- U10: value 74AHC1G08 -> 74ACHT132; footprint Package_TO_SOT_SMD:SOT-23-5_HandSoldering -> Package_SO:SOIC-14_3.9x8.7mm_P1.27mm; moved to F.Cu
- moved Q2 13.4 mm to (35.4, 111.0), turned to 0 degrees
- moved U9 5.24 mm to (44.5, 101.6)
- moved U10 5.17 mm to (34.2, 101.6), turned to 0 degrees
- moved C11 4.91 mm to (47.2, 95.2)
- moved J6 2.36 mm to (31.8, 116.0)
- moved C8 1.04 mm to (38.1, 91.4), turned to 180 degrees
Connections:
- U10 pad 1: /RUN -> /~STEP
- U10 pad 2: Net-(U9-1~{Q}) -> /~STEP
- U10 pad 3: GND -> Net-(U9-1CLK)
- U10 pad 4: Net-(U9-2~{PRE}) -> Net-(U9-1~{Q})
- U10 pad 5: +5V -> /RUN
- U9 pad 1: Net-(Q2-G) -> Net-(U9-1~{CLR})
- U9 pad 10: Net-(U9-2~{PRE}) -> +5V
- U9 pad 12: GND -> +5V
- U9 pad 13: +5V -> Net-(U9-2~{CLR})
- U9 pad 3: /~STEP -> Net-(U9-1CLK)
- U9 pad 8: Net-(Q2-G) -> Net-(U9-2~{Q})
- U9 pad 9: unconnected-(U9-2Q-Pad9) -> Net-(Q2-G)
Routing:
- net +5V: track 74.6 -> 94.8 mm
- net Net-(U9-2~{CLR}): track 0.00 -> 18.4 mm, vias 0 -> 2
- net Net-(U9-1~{CLR}): track 0.00 -> 12.9 mm, vias 0 -> 2
- net Net-(U9-2~{Q}): track 0.00 -> 12.4 mm
- net Net-(Q2-G): track 6.92 -> 19.2 mm
- net Net-(U9-1~{Q}): track 0.00 -> 11.9 mm
- net Net-(U9-1CLK): track 0.00 -> 10.8 mm
- net /~M1~: track 102.3 -> 111.0 mm
- net /~WAIT~: track 144.5 -> 136.1 mm
- net /~STEP: track 231.7 -> 225.0 mm
- net /RUN: track 217.7 -> 224.1 mm
- net Net-(U10-Pad10): track 0.00 -> 6.22 mm
- net /BUSAK: track 142.0 -> 143.0 mm
- net GND: track 337.0 -> 337.3 mm, vias 112 -> 113
