File: boards/Zx50_Cpu_RevC1/Zx50_Cpu_RevC1.kicad_sch (KiCad schematic)
At the start: 38 parts, among them J1 Zx50_EdgeConnector, J2 FrontPanelConnect, J3 Clock Mezzanine, J4 Front Panel, J5 TP_D_DIR, J6 TP_BUSAK, Q1 BSS84, Q2 2N7002-7-F, SW1 RESET, U1 74AHC1G14, U10 74ACHT132, U2 SN74ABT245BN, U3 SN74ABT245BN, U4 Z84C00xxP, U5 SN74ABT245BN, U6 MCP1316MT-46LE/OT, U7 SN74ABT245BN, U8 74LVC1G3208, U9 SN74AHCT74DRG4

Commit message: cpu revc1
Other:
- added sheet CoProcessor (coprocessor.kicad_sch)
Changed lines of the file:
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@@
 	(bus
 		(pts
+			(xy 83.82 237.49) (xy 87.63 237.49)
+		)
+		(stroke
+			(width 0)
+			(type default)
+		)
+	)
+	(bus
+		(pts
 			(xy 69.85 140.97) (xy 71.12 140.97)
 		)
@@
 	(bus
 		(pts
+			(xy 83.82 241.3) (xy 87.63 241.3)
+		)
+		(stroke
+			(width 0)
+			(type default)
+		)
+	)
+	(bus
+		(pts
 			(xy 102.87 88.9) (xy 105.41 88.9)
 		)
@@
 		)
 	)
+	(bus
+		(pts
+			(xy 83.82 229.87) (xy 87.63 229.87)
+		)
+		(stroke
+			(width 0)
+			(type default)
+		)
+	)
 	(wire
 		(pts
@@
 	(bus
 		(pts
+			(xy 83.82 233.68) (xy 87.63 233.68)
+		)
+		(stroke
+			(width 0)
+			(type default)
+		)
+	)
+	(bus
+		(pts
 			(xy 144.78 68.58) (xy 146.05 68.58)
 		)
@@
 		)
 	)
+	(label "{Z80_C}"
+		(at 83.82 237.49 180)
+		(effects
+			(font
+				(size 1.27 1.27)
+			)
+			(justify right bottom)
+		)
+	)
 	(label "A13"
 		(at 109.22 64.77 90)
@@
 		)
 	)
+	(label "{Z80_A}"
+		(at 83.82 229.87 180)
+		(effects
+			(font
+				(size 1.27 1.27)
+			)
+			(justify right bottom)
+		)
+	)
 	(label "~RFSH~"
 		(at 207.01 99.06 90)
@@
 		)
 	)
+	(label "{Z80_D}"
+		(at 83.82 233.68 180)
+		(effects
+			(font
+				(size 1.27 1.27)
+			)
+			(justify right bottom)
+		)
+	)
 	(label "BUS.D3"
 		(at 154.94 120.65 270)
@@
 		)
 	)
+	(label "{SH_C}"
+		(at 83.82 241.3 180)
+		(effects
+			(font
+				(size 1.27 1.27)
+			)
+			(justify right bottom)
+		)
+	)
 	(label "A6"
 		(at 127 64.7224 90)
@@
 		)
 		(instances
-			(project "Zx50_Cpu_RevB1"
+			(project "Zx50_Cpu_RevC1"
 				(path "/d27e6793-29e8-4553-aae0-c58a11de5d25"
 					(reference "C12")
@@
 		)
 		(instances
-			(project "Zx50_Cpu_RevB1"
+			(project "Zx50_Cpu_RevC1"
 				(path "/d27e6793-29e8-4553-aae0-c58a11de5d25"
 					(reference "#PWR045")
@@
 		)
 		(instances
-			(project "Zx50_Cpu_RevB1"
+			(project "Zx50_Cpu_RevC1"
 				(path "/d27e6793-29e8-4553-aae0-c58a11de5d25"
 					(reference "#PWR044")
@@
 				)
 			)
+		)
+	)
+	(sheet
+		(at 87.63 227.33)
+		(size 53.34 20.32)
+		(exclude_from_sim no)
+		(in_bom yes)
+		(on_board yes)
+		(dnp no)
+		(fields_autoplaced yes)
+		(stroke
+			(width 0.1524)
+			(type solid)
+		)
+		(fill
+			(color 0 0 0 0.0000)
+		)
+		(property "Sheetname" "CoProcessor"
+			(at 87.63 226.6184 0)
+			(effects
+				(font
+					(size 1.27 1.27)
+				)
+				(justify left bottom)
+			)
+		)
+		(property "Sheetfile" "coprocessor.kicad_sch"
+			(at 87.63 248.2346 0)
+			(effects
+				(font
+					(size 1.27 1.27)
+				)
+				(justify left top)
+			)
+		)
+		(pin "{Z80_D}" input
+			(at 87.63 233.68 180)
+			(effects
+				(font
+					(size 1.27 1.27)
+				)
+				(justify left)
+			)
+		)
+		(pin "{Z80_A}" input
+			(at 87.63 229.87 180)
+			(effects
+				(font
+					(size 1.27 1.27)
+				)
+				(justify left)
+			)
+		)
+		(pin "{Z80_C}" input
+			(at 87.63 237.49 180)
+			(effects
+				(font
+					(size 1.27 1.27)
+				)
+				(justify left)
+			)
+		)
+		(pin "{SH_C}" input
+			(at 87.63 241.3 180)
+			(effects
+				(font
+					(size 1.27 1.27)
+				)
+				(justify left)
+			)
+		)
+		(instances
+			(project "Zx50_Cpu_RevC1"
+				(path "/d27e6793-29e8-4553-aae0-c58a11de5d25"
+					(page "2")
+				)
+			)
