File: boards/Zx50_Cpu_RevC1/Zx50_Cpu_RevC1.kicad_pcb (KiCad board)
At the start: 6 copper layers, 133.5 x 100.3 mm, 57 parts, among them J1 Zx50_EdgeConnector, J2 FrontPanelConnect, J3 Clock Mezzanine, J4 Front Panel, J5 TP_D_DIR, J6 TP_BUSAK, J7 Conn_01x06_Pin, Q1 BSS84, Q2 2N7002-7-F, SW1 RESET, U1 74AHC1G14, U10 74ACHT132, U11 ATF1508ASx-xxJx84, U12 IS61C5128AS-25QLI, U13 SST39SF040, U2 SN74ABT245BN, U3 SN74ABT245BN, U4 Z84C00xxP, U5 SN74ABT245BN, U6 MCP1316MT-46LE/OT, U7 SN74ABT245BN, U8 74LVC1G3208, U9 SN74AHCT74DRG4

Commit message: init tb now runs against fpu
Parts:
- added J8: MEM SPD, Connector_PinHeader_2.54mm:PinHeader_1x02_P2.54mm_Vertical, F.Cu at (146.1, 142.9)
- added R5: 10K, Resistor_SMD:R_0805_2012Metric_Pad1.20x1.40mm_HandSolder, F.Cu at (151.8, 157.8)
- J7: value Conn_01x06_Pin -> JTAG
- moved J2 2.84 mm to (142.9, 153.7)
Connections:
- U11 pad 81: unconnected-(U11-I/O/GCLK3-Pad81) -> /CoProcessor/CLK_SPD
Routing:
- net /CoProcessor/CLK_SPD: track 0.00 -> 38.8 mm
- net Net-(J1-GPIO15): track 7.67 -> 5.34 mm
- net Net-(J1-AUX): track 11.3 -> 8.94 mm
- net /~WAIT~: track 249.1 -> 251.3 mm
- net +5V: track 192.3 -> 194.1 mm, vias 31 -> 32
Other:
- board text added: "+5V"
- board text added: "CLK SPD"
- board text added: "Zx50 CPU + FPU Modular Clock Marc Mosko, 2026 Zx50_Cpu_RevC.1"
- board text removed: "+5"
- board text removed: "Zx50 CPU Modular Clock Marc Mosko, 2026 Zx50_Cpu_RevB.1"
