File: boards/legacy/Zx50_Cpu_RevC2/coprocessor.kicad_sch (KiCad schematic)
At the start: 19 parts, among them J7 JTAG, J8 MEM SPD, U11 ATF1508ASx-xxJx84, U12 IS61C256AL-12TLI, U13 SST39SF040

Commit message: scrap the cpld, go fpga.  starting to rewrite the FPU architecture documents.
Parts:
- renumbered C24 to C?, C18 to C?, C23 to C?, C20 to C?, C22 to C?, C19 to C?, C14 to C?, C16 to C?, C17 to C?, C15 to C?, C21 to C?, J7 to J?, J8 to J?, R10 to R?, R7 to R?, R5 to R?, U11 to U?, U13 to U?, U12 to U?
Changed lines of the file:
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@@
 		(dnp no)
 		(fields_autoplaced yes)
-		(property "Reference" "#PWR054"
+		(property "Reference" "#PWR?"
 			(at 128.27 154.94 0)
 			(effects
@@
 		(on_board yes)
 		(dnp no)
-		(property "Reference" "C24"
+		(property "Reference" "C?"
 			(at 116.84 157.4801 0)
 			(effects
@@
 		)
 		(instances
+			(project "coprocessor"
+				(path "/3570fc7f-dae7-47bf-90e6-c8479ed556cd"
+					(reference "C?")
+					(unit 1)
+				)
+			)
 			(project "Zx50_Cpu_RevC2"
 				(path "/d27e6793-29e8-4553-aae0-c58a11de5d25/b98b1677-4c21-433e-bc3e-64f5e8297f28"
@@
 		(dnp no)
 		(fields_autoplaced yes)
-		(property "Reference" "#PWR053"
+		(property "Reference" "#PWR?"
 			(at 208.28 154.94 0)
 			(effects
@@
 		(on_board yes)
 		(dnp no)
-		(property "Reference" "U11"
+		(property "Reference" "U?"
 			(at 70.358 146.304 0)
 			(effects
@@
 		(dnp no)
 		(fields_autoplaced yes)
-		(property "Reference" "#PWR056"
+		(property "Reference" "#PWR?"
 			(at 73.66 34.29 0)
 			(effects
@@
 		(dnp no)
 		(fields_autoplaced yes)
-		(property "Reference" "#PWR049"
+		(property "Reference" "#PWR?"
 			(at 157.48 80.01 0)
 			(effects
@@
 		(dnp no)
 		(fields_autoplaced yes)
-		(property "Reference" "#PWR050"
+		(property "Reference" "#PWR?"
 			(at 220.98 157.48 0)
 			(effects
@@
 		(dnp no)
 		(fields_autoplaced yes)
-		(property "Reference" "U13"
+		(property "Reference" "U?"
 			(at 223.1233 76.2 0)
 			(effects
@@
 		(on_board yes)
 		(dnp no)
-		(property "Reference" "C18"
+		(property "Reference" "C?"
 			(at 100.33 21.844 0)
 			(effects
@@
 		)
 		(instances
+			(project "coprocessor"
+				(path "/3570fc7f-dae7-47bf-90e6-c8479ed556cd"
+					(reference "C?")
+					(unit 1)
+				)
+			)
 			(project "Zx50_Cpu_RevC2"
 				(path "/d27e6793-29e8-4553-aae0-c58a11de5d25/b98b1677-4c21-433e-bc3e-64f5e8297f28"
@@
 		(on_board yes)
 		(dnp no)
-		(property "Reference" "C23"
+		(property "Reference" "C?"
 			(at 137.16 21.844 0)
 			(effects
@@
 		)
 		(instances
+			(project "coprocessor"
+				(path "/3570fc7f-dae7-47bf-90e6-c8479ed556cd"
+					(reference "C?")
+					(unit 1)
+				)
+			)
 			(project "Zx50_Cpu_RevC2"
 				(path "/d27e6793-29e8-4553-aae0-c58a11de5d25/b98b1677-4c21-433e-bc3e-64f5e8297f28"
@@
 		(dnp no)
 		(fields_autoplaced yes)
-		(property "Reference" "#PWR046"
+		(property "Reference" "#PWR?"
 			(at 220.98 71.12 0)
 			(effects
@@
 		(on_board yes)
 		(dnp no)
-		(property "Reference" "C20"
+		(property "Reference" "C?"
 			(at 115.57 21.844 0)
 			(effects
@@
 		)
 		(instances
+			(project "coprocessor"
+				(path "/3570fc7f-dae7-47bf-90e6-c8479ed556cd"
+					(reference "C?")
+					(unit 1)
+				)
+			)
 			(project "Zx50_Cpu_RevC2"
 				(path "/d27e6793-29e8-4553-aae0-c58a11de5d25/b98b1677-4c21-433e-bc3e-64f5e8297f28"
@@
 		(dnp no)
 		(fields_autoplaced yes)
-		(property "Reference" "#PWR058"
+		(property "Reference" "#PWR?"
 			(at 109.22 167.64 0)
 			(effects
@@
 		)
 		(instances
+			(project "coprocessor"
+				(path "/3570fc7f-dae7-47bf-90e6-c8479ed556cd"
+					(reference "#PWR?")
+					(unit 1)
+				)
+			)
 			(project "Zx50_Cpu_RevC2"
 				(path "/d27e6793-29e8-4553-aae0-c58a11de5d25/b98b1677-4c21-433e-bc3e-64f5e8297f28"
@@
 		(on_board yes)
 		(dnp no)
-		(property "Reference" "C22"
+		(property "Reference" "C?"
 			(at 129.54 21.844 0)
 			(effects
@@
 		)
 		(instances
+			(project "coprocessor"
+				(path "/3570fc7f-dae7-47bf-90e6-c8479ed556cd"
+					(reference "C?")
+					(unit 1)
+				)
+			)
 			(project "Zx50_Cpu_RevC2"
 				(path "/d27e6793-29e8-4553-aae0-c58a11de5d25/b98b1677-4c21-433e-bc3e-64f5e8297f28"
@@
 		(on_board yes)
 		(dnp no)
-		(property "Reference" "R10"
+		(property "Reference" "R?"
 			(at 203.962 154.432 0)
 			(effects
@@
 		(dnp no)
 		(fields_autoplaced yes)
-		(property "Reference" "#PWR051"
+		(property "Reference" "#PWR?"
 			(at 167.64 128.27 0)
 			(effects
@@
 		(on_board yes)
 		(dnp no)
-		(property "Reference" "C19"
+		(property "Reference" "C?"
 			(at 107.95 21.844 0)
 			(effects
@@
 		)
 		(instances
+			(project "coprocessor"
+				(path "/3570fc7f-dae7-47bf-90e6-c8479ed556cd"
+					(reference "C?")
+					(unit 1)
+				)
+			)
 			(project "Zx50_Cpu_RevC2"
 				(path "/d27e6793-29e8-4553-aae0-c58a11de5d25/b98b1677-4c21-433e-bc3e-64f5e8297f28"
@@
 		(on_board yes)
 		(dnp no)
-		(property "Reference" "C14"
+		(property "Reference" "C?"
 			(at 91.44 21.082 0)
 			(effects
@@
 		(dnp no)
 		(fields_autoplaced yes)
-		(property "Reference" "#PWR055"
+		(property "Reference" "#PWR?"
 			(at 68.58 38.1 0)
 			(effects
@@
 		(dnp no)
 		(fields_autoplaced yes)
-		(property "Reference" "#PWR060"
+		(property "Reference" "#PWR?"
 			(at 198.12 129.54 0)
 			(effects
@@
 		)
 		(instances
+			(project "coprocessor"
+				(path "/3570fc7f-dae7-47bf-90e6-c8479ed556cd"
+					(reference "#PWR?")
+					(unit 1)
+				)
+			)
 			(project "Zx50_Cpu_RevC2"
 				(path "/d27e6793-29e8-4553-aae0-c58a11de5d25/b98b1677-4c21-433e-bc3e-64f5e8297f28"
@@
 		(dnp no)
 		(fields_autoplaced yes)
-		(property "Reference" "#PWR048"
+		(property "Reference" "#PWR?"
 			(at 212.09 80.01 0)
 			(effects
@@
 		(on_board yes)
 		(dnp no)
-		(property "Reference" "C16"
+		(property "Reference" "C?"
 			(at 162.5599 67.31 0)
 			(effects
@@
 		(on_board yes)
 		(dnp no)
-		(property "Reference" "C17"
+		(property "Reference" "C?"
 			(at 215.8999 67.31 0)
 			(effects
@@
 		(dnp no)
 		(fields_autoplaced yes)
-		(property "Reference" "#PWR047"
+		(property "Reference" "#PWR?"
 			(at 167.64 71.12 0)
 			(effects
@@
 		(on_board yes)
 		(dnp no)
-		(property "Reference" "R7"
+		(property "Reference" "R?"
 			(at 181.102 69.088 0)
 			(effects
@@
 		(on_board yes)
 		(dnp no)
-		(property "Reference" "C15"
+		(property "Reference" "C?"
 			(at 149.86 30.6069 0)
 			(effects
@@
 		(dnp no)
 		(fields_autoplaced yes)
-		(property "Reference" "#PWR052"
+		(property "Reference" "#PWR?"
 			(at 86.36 157.48 0)
 			(effects
@@
 		(on_board yes)
 		(dnp no)
-		(property "Reference" "C21"
+		(property "Reference" "C?"
 			(at 123.19 21.844 0)
 			(effects
@@
 		)
 		(instances
+			(project "coprocessor"
+				(path "/3570fc7f-dae7-47bf-90e6-c8479ed556cd"
+					(reference "C?")
+					(unit 1)
+				)
+			)
 			(project "Zx50_Cpu_RevC2"
 				(path "/d27e6793-29e8-4553-aae0-c58a11de5d25/b98b1677-4c21-433e-bc3e-64f5e8297f28"
@@
 		(dnp no)
 		(fields_autoplaced yes)
-		(property "Reference" "U12"
+		(property "Reference" "U?"
 			(at 166.37 74.93 0)
 			(effects
@@
 		)
 		(instances
+			(project "coprocessor"
+				(path "/3570fc7f-dae7-47bf-90e6-c8479ed556cd"
+					(reference "U?")
+					(unit 1)
+				)
+			)
 			(project ""
 				(path "/d27e6793-29e8-4553-aae0-c58a11de5d25/b98b1677-4c21-433e-bc3e-64f5e8297f28"
@@
 		(on_board yes)
 		(dnp no)
-		(property "Reference" "R5"
+		(property "Reference" "R?"
 			(at 104.902 154.432 0)
 			(effects
@@
 		)
 		(instances
+			(project "coprocessor"
+				(path "/3570fc7f-dae7-47bf-90e6-c8479ed556cd"
+					(reference "R?")
+					(unit 1)
+				)
+			)
 			(project "Zx50_Cpu_RevC2"
 				(path "/d27e6793-29e8-4553-aae0-c58a11de5d25/b98b1677-4c21-433e-bc3e-64f5e8297f28"
@@
 		(on_board yes)
 		(dnp no)
-		(property "Reference" "J7"
+		(property "Reference" "J?"
 			(at 120.65 145.796 0)
 			(effects
@@
 		)
 		(instances
+			(project "coprocessor"
+				(path "/3570fc7f-dae7-47bf-90e6-c8479ed556cd"
+					(reference "J?")
+					(unit 1)
+				)
+			)
 			(project ""
 				(path "/d27e6793-29e8-4553-aae0-c58a11de5d25/b98b1677-4c21-433e-bc3e-64f5e8297f28"
@@
 		(on_board yes)
 		(dnp no)
-		(property "Reference" "J8"
+		(property "Reference" "J?"
 			(at 120.65 125.7299 0)
 			(effects
@@
 		)
 		(instances
+			(project "coprocessor"
+				(path "/3570fc7f-dae7-47bf-90e6-c8479ed556cd"
+					(reference "J?")
+					(unit 1)
+				)
+			)
 			(project ""
 				(path "/d27e6793-29e8-4553-aae0-c58a11de5d25/b98b1677-4c21-433e-bc3e-64f5e8297f28"
